File: MCU Datalogger.kicad_sch (KiCad schematic)
At the start: 25 parts, among them U1 24LC1025, U2 DS1337S+, U3 24LC1025, U4 ATMEGA328-AU, Y1 32.768KHz, Y2 16MHz

Commit message: comments
Other:
- note added: "EEPROM Memory"
- note added: "MCU"
- note added: "Mounting"
- note added: "Real Time Clock"
Changed lines of the file:
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@@
+    (stroke (width 0) (type default) (color 0 0 0 0))
+  )
+  (polyline (pts (xy 173.99 111.76) (xy 203.2 111.76))
+    (stroke (width 0) (type default) (color 0 0 0 0))
+  )
+  (polyline (pts (xy 133.35 165.1) (xy 133.35 127))
     (stroke (width 0) (type default) (color 0 0 0 0))
   )
@@
     (stroke (width 0) (type default) (color 0 0 0 0))
   )
+  (polyline (pts (xy 149.86 20.32) (xy 279.4 20.32))
+    (stroke (width 0) (type default) (color 0 0 0 0))
+  )
   (wire (pts (xy 119.38 138.43) (xy 124.46 138.43))
     (stroke (width 0) (type default) (color 0 0 0 0))
@@
     (stroke (width 0) (type default) (color 0 0 0 0))
   )
+  (polyline (pts (xy 173.99 111.76) (xy 173.99 149.86))
+    (stroke (width 0) (type default) (color 0 0 0 0))
+  )
   (wire (pts (xy 227.33 80.01) (xy 227.33 82.55))
     (stroke (width 0) (type default) (color 0 0 0 0))
@@
     (stroke (width 0) (type default) (color 0 0 0 0))
   )
+  (polyline (pts (xy 173.99 149.86) (xy 203.2 149.86))
+    (stroke (width 0) (type default) (color 0 0 0 0))
+  )
   (wire (pts (xy 177.8 54.61) (xy 177.8 53.34))
     (stroke (width 0) (type default) (color 0 0 0 0))
   )
+  (polyline (pts (xy 35.56 127) (xy 133.35 127))
+    (stroke (width 0) (type default) (color 0 0 0 0))
+  )
   (wire (pts (xy 92.71 148.59) (xy 92.71 154.94))
     (stroke (width 0) (type default) (color 0 0 0 0))
@@
     (stroke (width 0) (type default) (color 0 0 0 0))
   )
+  (polyline (pts (xy 124.46 36.83) (xy 124.46 86.36))
+    (stroke (width 0) (type default) (color 0 0 0 0))
+  )
   (wire (pts (xy 252.73 31.75) (xy 266.7 31.75))
     (stroke (width 0) (type default) (color 0 0 0 0))
@@
     (stroke (width 0) (type default) (color 0 0 0 0))
   )
+  (polyline (pts (xy 149.86 20.32) (xy 149.86 93.98))
+    (stroke (width 0) (type default) (color 0 0 0 0))
+  )
   (wire (pts (xy 166.37 46.99) (xy 168.91 46.99))
     (stroke (width 0) (type default) (color 0 0 0 0))
@@
     (stroke (width 0) (type default) (color 0 0 0 0))
   )
+  (polyline (pts (xy 203.2 149.86) (xy 203.2 111.76))
+    (stroke (width 0) (type default) (color 0 0 0 0))
+  )
   (wire (pts (xy 163.83 53.34) (xy 177.8 53.34))
     (stroke (width 0) (type default) (color 0 0 0 0))
@@
     (stroke (width 0) (type default) (color 0 0 0 0))
   )
+  (polyline (pts (xy 149.86 93.98) (xy 279.4 93.98))
+    (stroke (width 0) (type default) (color 0 0 0 0))
+  )
   (wire (pts (xy 83.82 50.8) (xy 90.17 50.8))
     (stroke (width 0) (type default) (color 0 0 0 0))
@@
     (stroke (width 0) (type default) (color 0 0 0 0))
   )
+  (polyline (pts (xy 279.4 93.98) (xy 279.4 20.32))
+    (stroke (width 0) (type default) (color 0 0 0 0))
+  )
   (wire (pts (xy 182.88 54.61) (xy 182.88 53.34))
     (stroke (width 0) (type default) (color 0 0 0 0))
@@
     (stroke (width 0) (type default) (color 0 0 0 0))
   )
+  (polyline (pts (xy 35.56 127) (xy 35.56 165.1))
+    (stroke (width 0) (type default) (color 0 0 0 0))
+  )
   (wire (pts (xy 88.9 55.88) (xy 83.82 55.88))
     (stroke (width 0) (type default) (color 0 0 0 0))
   )
+  (polyline (pts (xy 124.46 86.36) (xy 25.4 86.36))
+    (stroke (width 0) (type default) (color 0 0 0 0))
+  )
   (wire (pts (xy 196.85 54.61) (xy 182.88 54.61))
     (stroke (width 0) (type default) (color 0 0 0 0))
   )
+  (polyline (pts (xy 25.4 36.83) (xy 25.4 86.36))
+    (stroke (width 0) (type default) (color 0 0 0 0))
+  )
   (wire (pts (xy 95.25 44.45) (xy 95.25 50.8))
     (stroke (width 0) (type default) (color 0 0 0 0))
@@
     (stroke (width 0) (type default) (color 0 0 0 0))
   )
+  (polyline (pts (xy 35.56 165.1) (xy 133.35 165.1))
+    (stroke (width 0) (type default) (color 0 0 0 0))
+  )
   (wire (pts (xy 87.63 73.66) (xy 87.63 76.2))
     (stroke (width 0) (type default) (color 0 0 0 0))
   )
+  (polyline (pts (xy 25.4 36.83) (xy 124.46 36.83))
+    (stroke (width 0) (type default) (color 0 0 0 0))
+  )
   (wire (pts (xy 106.68 59.69) (xy 83.82 59.69))
     (stroke (width 0) (type default) (color 0 0 0 0))
@@
     (stroke (width 0) (type default) (color 0 0 0 0))
   )
+  (text "EEPROM Memory" (at 68.58 127 0)
+    (effects (font (size 1.27 1.27)) (justify left bottom))
+  )
+  (text "Mounting" (at 179.07 111.76 0)
+    (effects (font (size 1.27 1.27)) (justify left bottom))
+  )
+  (text "Real Time Clock\n" (at 39.37 36.83 0)
+    (effects (font (size 1.27 1.27)) (justify left bottom))
+  )
+  (text "MCU\n" (at 185.42 20.32 0)
+    (effects (font (size 1.27 1.27)) (justify left bottom))
+  )
   (label "SCK" (at 92.71 146.05 0)

Commit message: setup pcbnew
Parts:
- U2: footprint SOIC127P600X175-8N -> digikey-footprints:SOIC127P600X175-8N
- U4: footprint QFP80P900X900X120-32N -> digikey-footprints:QFP80P900X900X120-32N
Changed lines of the file:
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@@
     (property "Reference" "U2" (id 0) (at 66.04 44.2173 0))
     (property "Value" "DS1337S+" (id 1) (at 66.04 46.9924 0))
-    (property "Footprint" "SOIC127P600X175-8N" (id 2) (at 66.04 63.5 0)
+    (property "Footprint" "digikey-footprints:SOIC127P600X175-8N" (id 2) (at 66.04 63.5 0)
       (effects (font (size 1.27 1.27)) (justify left bottom) hide)
     )
@@
     (property "Reference" "U4" (id 0) (at 212.09 25.2435 0))
     (property "Value" "ATMEGA328-AU" (id 1) (at 212.09 28.0186 0))
-    (property "Footprint" "QFP80P900X900X120-32N" (id 2) (at 212.09 57.15 0)
+    (property "Footprint" "digikey-footprints:QFP80P900X900X120-32N" (id 2) (at 212.09 57.15 0)
       (effects (font (size 1.27 1.27)) (justify left bottom) hide)
     )
@@
     )
     (path "/19c98a84-20a8-4af9-9cc1-9d31e850c8dd"
-      (reference "U2") (unit 1) (value "DS1337S+") (footprint "SOIC127P600X175-8N")
+      (reference "U2") (unit 1) (value "DS1337S+") (footprint "digikey-footprints:SOIC127P600X175-8N")
     )
     (path "/34ab20fe-5be7-4a63-8a85-5703b7882acf"
@@
     )
     (path "/25d9e195-a4aa-413a-8272-cdbb8630ad4f"
-      (reference "U4") (unit 1) (value "ATMEGA328-AU") (footprint "QFP80P900X900X120-32N")
+      (reference "U4") (unit 1) (value "ATMEGA328-AU") (footprint "digikey-footprints:QFP80P900X900X120-32N")
     )
     (path "/a107f895-390a-45c8-b926-bb94c406e415"
