File: MCU Datalogger.kicad_sch (KiCad schematic)
At the start: 25 parts, among them U1 24LC1025, U2 DS1337S+, U3 24LC1025, U4 ATMEGA328-AU, Y1 32.768KHz, Y2 16MHz

Commit message: PCB footprint placement
Parts:
- BT1: footprint Connector_PinHeader_2.54mm:PinHeader_1x02_P2.54mm_Horizontal -> Connector_PinHeader_2.54mm:PinHeader_1x02_P2.54mm_Vertical
Changed lines of the file:
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@@
       (effects (font (size 1.27 1.27)) (justify left))
     )
-    (property "Footprint" "Connector_PinHeader_2.54mm:PinHeader_1x02_P2.54mm_Horizontal" (id 2) (at 266.7 35.306 90)
+    (property "Footprint" "Connector_PinHeader_2.54mm:PinHeader_1x02_P2.54mm_Vertical" (id 2) (at 266.7 35.306 90)
       (effects (font (size 1.27 1.27)) hide)
     )
@@
     )
     (path "/9024e82c-4898-4285-8617-60ba26442fd0"
-      (reference "BT1") (unit 1) (value "Battery") (footprint "Connector_PinHeader_2.54mm:PinHeader_1x02_P2.54mm_Horizontal")
+      (reference "BT1") (unit 1) (value "Battery") (footprint "Connector_PinHeader_2.54mm:PinHeader_1x02_P2.54mm_Vertical")
     )
     (path "/76acfa45-f969-4555-894c-92213c0bf6ef"

Commit message: rooting
Connections:
- net Vcc: now also R3.1, R4.1
Changed lines of the file:
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@@
+    (stroke (width 0) (type default) (color 0 0 0 0))
+  )
+  (wire (pts (xy 166.37 48.26) (xy 166.37 46.99))
     (stroke (width 0) (type default) (color 0 0 0 0))
   )
@@
     (effects (font (size 1.27 1.27)) (justify right bottom))
   )
+  (label "Vcc" (at 119.38 133.35 0)
+    (effects (font (size 1.27 1.27)) (justify left bottom))
+  )
   (label "Vcc" (at 222.25 110.49 180)
     (effects (font (size 1.27 1.27)) (justify right bottom))
@@
     (effects (font (size 1.27 1.27)) (justify right bottom))
   )
+  (label "D2" (at 260.35 107.95 0)
+    (effects (font (size 1.27 1.27)) (justify left bottom))
+  )
+  (label "Vcc" (at 167.64 77.47 0)
+    (effects (font (size 1.27 1.27)) (justify left bottom))
+  )
+  (label "D8" (at 260.35 123.19 0)
+    (effects (font (size 1.27 1.27)) (justify left bottom))
+  )
+  (label "D6" (at 260.35 118.11 0)
+    (effects (font (size 1.27 1.27)) (justify left bottom))
+  )
+  (label "SCK" (at 196.85 52.07 180)
+    (effects (font (size 1.27 1.27)) (justify right bottom))
+  )
+  (label "D4" (at 260.35 113.03 0)
+    (effects (font (size 1.27 1.27)) (justify left bottom))
+  )
+  (label "RESET" (at 229.87 144.78 180)
+    (effects (font (size 1.27 1.27)) (justify right bottom))
+  )
+  (label "MOSI" (at 196.85 46.99 180)
+    (effects (font (size 1.27 1.27)) (justify right bottom))
+  )
+  (label "D7" (at 260.35 120.65 0)
+    (effects (font (size 1.27 1.27)) (justify left bottom))
+  )
+  (label "SCK" (at 229.87 129.54 180)
+    (effects (font (size 1.27 1.27)) (justify right bottom))
+  )
   (label "Vcc" (at 82.55 137.16 0)
     (effects (font (size 1.27 1.27)) (justify left bottom))
   )
-  (label "D2" (at 260.35 107.95 0)
-    (effects (font (size 1.27 1.27)) (justify left bottom))
-  )
-  (label "Vcc" (at 167.64 77.47 0)
-    (effects (font (size 1.27 1.27)) (justify left bottom))
-  )
-  (label "D8" (at 260.35 123.19 0)
-    (effects (font (size 1.27 1.27)) (justify left bottom))
-  )
-  (label "D6" (at 260.35 118.11 0)
-    (effects (font (size 1.27 1.27)) (justify left bottom))
-  )
-  (label "SCK" (at 196.85 52.07 180)
-    (effects (font (size 1.27 1.27)) (justify right bottom))
+  (label "SDA" (at 124.46 151.13 0)
+    (effects (font (size 1.27 1.27)) (justify left bottom))
   )
   (label "Vcc" (at 53.34 137.16 0)
-    (effects (font (size 1.27 1.27)) (justify left bottom))
-  )
-  (label "D4" (at 260.35 113.03 0)
-    (effects (font (size 1.27 1.27)) (justify left bottom))
-  )
-  (label "RESET" (at 229.87 144.78 180)
-    (effects (font (size 1.27 1.27)) (justify right bottom))
-  )
-  (label "MOSI" (at 196.85 46.99 180)
-    (effects (font (size 1.27 1.27)) (justify right bottom))
-  )
-  (label "D7" (at 260.35 120.65 0)
-    (effects (font (size 1.27 1.27)) (justify left bottom))
-  )
-  (label "SCK" (at 229.87 129.54 180)
-    (effects (font (size 1.27 1.27)) (justify right bottom))
-  )
-  (label "SDA" (at 124.46 151.13 0)
     (effects (font (size 1.27 1.27)) (justify left bottom))
   )
@@
     )
   )
-  (symbol (lib_id "power:GND") (at 166.37 46.99 0) (unit 1)
-    (in_bom yes) (on_board yes) (fields_autoplaced)
-    (property "Reference" "#PWR0109" (id 0) (at 166.37 53.34 0)
-      (effects (font (size 1.27 1.27)) hide)
-    )
-    (property "Value" "GND" (id 1) (at 166.37 51.5525 0))
-    (property "Footprint" "" (id 2) (at 166.37 46.99 0)
-      (effects (font (size 1.27 1.27)) hide)
-    )
-    (property "Datasheet" "" (id 3) (at 166.37 46.99 0)
-      (effects (font (size 1.27 1.27)) hide)
-    )
+  (symbol (lib_id "power:GND") (at 166.37 48.26 0) (unit 1)
+    (in_bom yes) (on_board yes) (fields_autoplaced)
+    (property "Reference" "#PWR0109" (id 0) (at 166.37 54.61 0)
+      (effects (font (size 1.27 1.27)) hide)
+    )
+    (property "Value" "GND" (id 1) (at 166.37 52.8225 0))
+    (property "Footprint" "" (id 2) (at 166.37 48.26 0)
+      (effects (font (size 1.27 1.27)) hide)
+    )
+    (property "Datasheet" "" (id 3) (at 166.37 48.26 0)
+      (effects (font (size 1.27 1.27)) hide)
+    )
